File: pcb/CocoMEMJr_v1.01.sch (EAGLE design)
At the start: 37 parts, among them IC1 CPU, IC2 HDR, IC3 XC95144XLTQG144, IC8 AZ1117CH-3.3

Commit message: Simplify the design for debugging
Parts:
- IC1, IC2: device micro-motorola:6809ER -> micro-motorola:MC6809ER
Changed lines of the file:
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@@
 <part name="SUPPLY3" library="supply2" deviceset="GND" device=""/>
 <part name="SUPPLY4" library="supply2" deviceset="VCC" device=""/>
-<part name="IC1" library="micro-motorola" deviceset="6809E" device="R" value="CPU"/>
-<part name="IC2" library="micro-motorola" deviceset="6809E" device="R" value="HDR"/>
+<part name="IC1" library="micro-motorola" deviceset="MC6809E" device="R" value="CPU"/>
+<part name="IC2" library="micro-motorola" deviceset="MC6809E" device="R" value="HDR"/>
 <part name="FRAME3" library="frames" deviceset="DINA3_L" device=""/>
 <part name="TDI" library="testpad" deviceset="TP" device="TP08R"/>
